Commit message: adjust the camera location

File: urdf/test.xacro (robot description, xacro)
@@ -3,11 +3,12 @@
   <xacro:include filename="$(find realsense_ros_gazebo)/xacro/tracker.xacro"/>
   <xacro:include filename="$(find realsense_ros_gazebo)/xacro/depthcam.xacro"/>
-  <link name="base_footprint"/>
+  <link name="world" />
+  <!-- <link name="base_footprint"/>
   <joint name="footprint_joint" type="fixed">
     <parent link="base_footprint"/>
     <child link="base_link"/>
     <origin rpy="0 0 0" xyz="0 0 0"/>
-  </joint>
-  <link name="base_link">
+  </joint> -->
+  <!-- <link name="base_link">
     <visual>
       <origin rpy="0 0 0 " xyz="0 0 0.005"/>
@@ -30,7 +31,7 @@
       <inertia ixx="1.0265" ixy="0" ixz="0" iyy="1.3944999999999999" iyz="0" izz="2.1320000000000001"/>
     </inertial>
-  </link>
+  </link> -->
   <!-- TEST -->
-  <xacro:realsense_d435 sensor_name="d435" parent_link="base_link" rate="10">
+  <xacro:realsense_d435 sensor_name="d435" parent_link="world" rate="10">
     <origin rpy="0 1.57 0 " xyz="0 0 2.0"/>
   </xacro:realsense_d435>
